File: v1/qrng.kicad_pcb (KiCad board)
At the start: 2 copper layers, 44 x 20.5 mm, 28 parts, among them J1 USB_A, U1 AMS1117, U2 STM32F103C8Tx, U3 W25N01GV, Y1 Crystal

Commit message: Separated ADC pins per recommendation from Epilogis
Parts:
- removed R1: R_Small, Resistor_SMD:R_0402_1005Metric
- added R4: 270, Resistor_SMD:R_0603_1608Metric, F.Cu at (150.1, 104.3)
- added R5: 100, Resistor_SMD:R_0603_1608Metric, F.Cu at (150.1, 101.2)
- C12, C13: value C_Small -> 30pF; footprint Capacitor_SMD:C_0402_1005Metric -> Capacitor_SMD:C_0603_1608Metric
- Y1: value Crystal -> 8 MHz
- moved C13 53.3 mm to (152.9, 108.2), turned to 90 degrees
- moved C6 48.5 mm to (135.8, 94.5)
- moved BS1 48.5 mm to (156.8, 100.2)
- moved C1 48.5 mm to (144.1, 104.5)
- moved C10 48.5 mm to (145.5, 93.9)
- moved C11 48.5 mm to (146.7, 98.0)
- moved C2 48.5 mm to (145.1, 104.5)
- moved C4 48.5 mm to (135.7, 103.0)
- moved C7 48.5 mm to (135.7, 104.1)
- moved C8 48.5 mm to (135.4, 99.8)
- moved C9 48.5 mm to (145.3, 99.8)
- moved D1 48.5 mm to (134.1, 94.2)
- moved D2 48.5 mm to (156.8, 108.5)
- moved FB1 48.5 mm to (134.9, 97.1)
- moved H1 48.5 mm to (161.5, 108.0)
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Connections:
- C13 pad 2: OSC_OUT -> Net-(C13-Pad2)
- U2 pad 10: Net-(U2-Pad10) -> (no net)
- U2 pad 13: Net-(U2-Pad13) -> (no net)
- U2 pad 15: Net-(U2-Pad15) -> (no net)
- U2 pad 16: Net-(U2-Pad16) -> (no net)
- U2 pad 17: Net-(U2-Pad17) -> (no net)
- U2 pad 18: Net-(U2-Pad18) -> (no net)
- U2 pad 19: Net-(U2-Pad19) -> (no net)
- U2 pad 2: Net-(U2-Pad2) -> (no net)
- U2 pad 20: Net-(U2-Pad20) -> (no net)
- U2 pad 21: Net-(U2-Pad21) -> (no net)
- U2 pad 22: Net-(U2-Pad22) -> (no net)
- U2 pad 29: Net-(U2-Pad29) -> (no net)
- U2 pad 3: Net-(U2-Pad3) -> (no net)
- U2 pad 30: Net-(U2-Pad30) -> (no net)
- U2 pad 31: Net-(U2-Pad31) -> (no net)
- U2 pad 38: Net-(U2-Pad38) -> (no net)
- U2 pad 4: Net-(U2-Pad4) -> (no net)
- U2 pad 40: Net-(U2-Pad40) -> (no net)
- U2 pad 41: Net-(U2-Pad41) -> (no net)
- U2 pad 42: Net-(U2-Pad42) -> (no net)
- U2 pad 43: Net-(U2-Pad43) -> (no net)
- U2 pad 44: BOOT0 -> (no net)
- U2 pad 45: Net-(U2-Pad45) -> (no net)
- U2 pad 46: Net-(U2-Pad46) -> (no net)
- U2 pad 7: NRST -> (no net)
- Y1 pad 2: Net-(R1-Pad1) -> Net-(C13-Pad2)
Routing:
- net OSC_IN: track 7.37 -> 16.1 mm
- net Net-(C13-Pad2): track 0.00 -> 6.26 mm
- net GND: track 34.7 -> 39.0 mm, vias 7 -> 9
- net OSC_OUT: track 3.02 -> 6.63 mm
- net Net-(R1-Pad1): track 3.17 -> 0.00 mm
- net +3V3: track 82.6 -> 79.6 mm, vias 5 -> 4
- net Net-(R4-Pad2): track 0.00 -> 1.97 mm
