File: v1/qrng.sch (KiCad schematic (older format))
At the start: 25 parts, among them J1 USB_A, J2 Conn_01x03, U1 AMS1117, U2 STM32F103C8Tx, U3 W25N01GV, Y1 Crystal

Commit message: Separated ADC pins per recommendation from Epilogis
Parts:
- removed R1: R_Small, Resistor_SMD:R_0402_1005Metric, symbol Device:R_Small
- added R4: 270, Resistor_SMD:R_0603_1608Metric, symbol Device:R_Small_US
- added R5: 100, Resistor_SMD:R_0603_1608Metric, symbol Device:R_Small_US
- C12, C13: value C_Small -> 30pF; footprint Capacitor_SMD:C_0402_1005Metric -> Capacitor_SMD:C_0603_1608Metric
- Y1: value Crystal -> 8 MHz
Other:
- moved on the sheet: C10, C11, C12, C13, FB2, H1, H2, J2, U2, U3, Y1
